File: pcb/muse.kicad_pcb (KiCad board)
At the start: 2 copper layers, 79.5 x 47 mm, 9 parts, among them J1 Conn_01x04, SW1 RotaryEncoder, SW2 SW_Push, SW3 SW_Push, SW4 SW_Push, SW5 SW_Push, SW6 SW_Push, SW7 SW_Push, U1 XIAO-RP2040-SMD

Commit message: Update footprint
Parts:
- U1: value XIAO-RP2040-SMD -> XIAO-RP2040
Changed lines of the file:
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@@
 		(sheetname "/")
 		(sheetfile "muse.kicad_sch")
-		(units
-			(unit
-				(name "A")
-				(pins "1" "2")
-			)
-		)
 		(attr through_hole)
 		(duplicate_pad_numbers_are_jumpers no)
@@
 		(sheetname "/")
 		(sheetfile "muse.kicad_sch")
-		(units
-			(unit
-				(name "A")
-				(pins "1" "2")
-			)
-		)
 		(attr smd)
 		(duplicate_pad_numbers_are_jumpers no)
@@
 		(sheetname "/")
 		(sheetfile "muse.kicad_sch")
-		(units
-			(unit
-				(name "A")
-				(pins "1" "2")
-			)
-		)
 		(attr through_hole)
 		(duplicate_pad_numbers_are_jumpers no)
@@
 		(sheetname "/")
 		(sheetfile "muse.kicad_sch")
-		(units
-			(unit
-				(name "A")
-				(pins "A" "C" "B")
-			)
-		)
 		(attr through_hole)
 		(duplicate_pad_numbers_are_jumpers no)
@@
 		)
 		(pad "1" smd rect
-			(at -5 7.9)
-			(size 2.5 3.2)
+			(at -5.125 7.9)
+			(size 2.25 3.2)
 			(layers "F.Cu" "F.Mask" "F.Paste")
 		)
 		(pad "2" smd rect
-			(at 5 7.9)
-			(size 2.5 3.2)
+			(at 5.125 7.9)
+			(size 2.25 3.2)
 			(layers "F.Cu" "F.Mask" "F.Paste")
 		)
@@
 		(sheetname "/")
 		(sheetfile "muse.kicad_sch")
-		(units
-			(unit
-				(name "A")
-				(pins "1" "2")
-			)
-		)
 		(attr through_hole)
 		(duplicate_pad_numbers_are_jumpers no)
@@
 		(sheetname "/")
 		(sheetfile "muse.kicad_sch")
-		(units
-			(unit
-				(name "A")
-				(pins "1" "2")
-			)
-		)
 		(attr through_hole)
 		(duplicate_pad_numbers_are_jumpers no)
@@
 		(sheetname "/")
 		(sheetfile "muse.kicad_sch")
-		(units
-			(unit
-				(name "A")
-				(pins "1" "2")
-			)
-		)
 		(attr through_hole)
 		(duplicate_pad_numbers_are_jumpers no)
@@
 		(sheetname "/")
 		(sheetfile "muse.kicad_sch")
-		(units
-			(unit
-				(name "A")
-				(pins "1" "2" "3" "4")
-			)
-		)
 		(attr through_hole)
 		(duplicate_pad_numbers_are_jumpers no)
@@
 		(layer "B.Cu")
 		(at 137.0805 102.338 180)
-		(property "Value" "XIAO-RP2040-SMD"
+		(property "Reference" "U1"
+			(at 8.0805 11.336 0)
+			(layer "B.SilkS")
+			(effects
+				(font
+					(size 0.8 0.8)
+					(thickness 0.1)
+				)
+				(justify left bottom mirror)
+			)
+		)
+		(property "Value" "XIAO-RP2040"
 			(at 8.89 10.795 0)
 			(layer "B.Fab")
@@
 			)
 		)
-		(property "Reference" "U1"
-			(at 8.0805 11.336 0)
-			(layer "B.SilkS")
-			(effects
-				(font
-					(size 0.8 0.8)
-					(thickness 0.1)
-				)
-				(justify left bottom mirror)
-			)
-		)
 		(sheetname "/")
 		(sheetfile "muse.kicad_sch")
-		(units
-			(unit
-				(name "A")
-				(pins "1" "2" "3" "4" "5" "6" "7" "24" "25" "32" "26" "33" "27" "14"
-					"13" "12" "11" "10" "9" "8"
-				)
-			)
-		)
 		(duplicate_pad_numbers_are_jumpers no)
 		(fp_line

Commit message: Add logo
Parts:
- added G***: LOGO, LOGO, F.Cu at (122.0, 103.0)
