File: pcb/muse.kicad_pcb (KiCad board)
At the start: 2 copper layers, 79.5 x 47 mm, 10 parts, among them J1 Conn_01x04, SW1 RotaryEncoder, SW2 SW_Push, SW3 SW_Push, SW4 SW_Push, SW5 SW_Push, SW6 SW_Push, SW7 SW_Push, U1 XIAO-RP2040

Commit message: Align traces
Routing:
- net S: track 22.1 -> 19.6 mm
- net SDA: track 19.2 -> 20.2 mm
Changed lines of the file:
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@@
 	)
 	(segment
-		(start 100.8 123.25)
+		(start 100.55 123)
 		(end 99.8 122.25)
 		(width 0.2)
@@
 	)
 	(segment
+		(start 142.25 119)
+		(end 138.25 123)
+		(width 0.2)
+		(layer "B.Cu")
+		(net "T1")
+	)
+	(segment
 		(start 146.799265 114.450735)
-		(end 136.2455 103.89697)
-		(width 0.2)
-		(layer "B.Cu")
-		(net "T1")
-	)
-	(segment
-		(start 138 123.25)
-		(end 100.8 123.25)
-		(width 0.2)
-		(layer "B.Cu")
-		(net "T1")
-	)
-	(segment
-		(start 142.25 119)
-		(end 138 123.25)
-		(width 0.2)
-		(layer "B.Cu")
-		(net "T1")
-	)
-	(segment
-		(start 136.2455 103.89697)
+		(end 146.516421 114.450735)
+		(width 0.2)
+		(layer "B.Cu")
+		(net "T1")
+	)
+	(segment
+		(start 138.25 123)
+		(end 100.55 123)
+		(width 0.2)
+		(layer "B.Cu")
+		(net "T1")
+	)
+	(segment
+		(start 146.516421 114.450735)
+		(end 136.2455 104.179814)
+		(width 0.2)
+		(layer "B.Cu")
+		(net "T1")
+	)
+	(segment
+		(start 136.2455 104.179814)
 		(end 136.2455 99.458)
 		(width 0.2)
@@
 	)
 	(segment
+		(start 124.75 94.25)
+		(end 123.5 94.25)
+		(width 0.2)
+		(layer "F.Cu")
+		(net "S")
+	)
+	(segment
 		(start 122.25 93)
 		(end 122.25 91.238)
@@
 		(net "S")
 	)
-	(segment
-		(start 124.75 94.25)
-		(end 123.5 94.25)
-		(width 0.2)
-		(layer "F.Cu")
-		(net "S")
-	)
 	(via
 		(at 122.25 91.238)
@@
 	)
 	(segment
-		(start 131.2935 94.25)
-		(end 126.75 94.25)
-		(width 0.2)
-		(layer "B.Cu")
-		(net "S")
-	)
-	(segment
-		(start 136.2455 89.298)
-		(end 131.2935 94.25)
+		(start 123.79 89.698)
+		(end 135.8455 89.698)
 		(width 0.2)
 		(layer "B.Cu")
@@
 	(segment
 		(start 122.25 91.238)
-		(end 123.738 91.238)
-		(width 0.2)
-		(layer "B.Cu")
-		(net "S")
-	)
-	(segment
-		(start 123.738 91.238)
-		(end 126.75 94.25)
+		(end 123.79 89.698)
+		(width 0.2)
+		(layer "B.Cu")
+		(net "S")
+	)
+	(segment
+		(start 135.8455 89.698)
+		(end 136.2455 89.298)
 		(width 0.2)
 		(layer "B.Cu")
@@
 	)
 	(segment
+		(start 117.477909 81.75)
+		(end 131.803186 81.75)
+		(width 0.2)
+		(layer "B.Cu")
+		(net "RA")
+	)
+	(segment
+		(start 131.803186 81.75)
+		(end 134.271186 84.218)
+		(width 0.2)
+		(layer "B.Cu")
+		(net "RA")
+	)
+	(segment
+		(start 100.375 98.852908)
+		(end 117.477909 81.75)
+		(width 0.2)
+		(layer "B.Cu")
+		(net "RA")
+	)
+	(segment
+		(start 134.271186 84.218)
+		(end 136.2455 84.218)
+		(width 0.2)
+		(layer "B.Cu")
+		(net "RA")
+	)
+	(segment
 		(start 100.375 99.5)
 		(end 100.375 98.852908)
@@
 	)
 	(segment
-		(start 100.375 98.852908)
-		(end 116.917908 82.31)
-		(width 0.2)
-		(layer "B.Cu")
-		(net "RA")
-	)
-	(segment
-		(start 116.917908 82.31)
-		(end 134.3375 82.31)
-		(width 0.2)
-		(layer "B.Cu")
-		(net "RA")
-	)
-	(segment
-		(start 134.3375 82.31)
-		(end 136.2455 84.218)
-		(width 0.2)
-		(layer "B.Cu")
-		(net "RA")
-	)
-	(segment
 		(start 105.375 99.5)
 		(end 105.375 101.55)
@@
 	)
 	(segment
-		(start 117.083594 82.71)
-		(end 105.375 94.418594)
-		(width 0.2)
-		(layer "B.Cu")
-		(net "RB")
-	)
-	(segment
-		(start 124.86 84.61)
-		(end 122.96 82.71)
-		(width 0.2)
-		(layer "B.Cu")
-		(net "RB")
-	)
-	(segment
-		(start 122.96 82.71)
-		(end 117.083594 82.71)
-		(width 0.2)
-		(layer "B.Cu")
-		(net "RB")
-	)
-	(segment
-		(start 136.2455 86.758)
-		(end 134.0975 84.61)
-		(width 0.2)
-		(layer "B.Cu")
-		(net "RB")
-	)
-	(segment
-		(start 134.0975 84.61)
-		(end 124.86 84.61)
-		(width 0.2)
-		(layer "B.Cu")
-		(net "RB")
-	)
-	(segment
 		(start 105.375 94.418594)
 		(end 105.375 99.5)
@@
 	)
 	(segment
+		(start 117.643594 82.15)
+		(end 105.375 94.418594)
+		(width 0.2)
+		(layer "B.Cu")
+		(net "RB")
+	)
+	(segment
+		(start 131.6375 82.15)
+		(end 117.643594 82.15)
+		(width 0.2)
+		(layer "B.Cu")
+		(net "RB")
+	)
+	(segment
+		(start 136.2455 86.758)
+		(end 131.6375 82.15)
+		(width 0.2)
+		(layer "B.Cu")
+		(net "RB")
+	)
+	(segment
 		(start 115.2875 122.25)
 		(end 115.2875 124.25)
@@
 	)
 	(segment
-		(start 128.25 119.725)
-		(end 128.25 105.0875)
+		(start 126 117.475)
+		(end 126 102.8375)
 		(width 0.2)
 		(layer "B.Cu")
@@
 	)
 	(segment
-		(start 128.25 105.0875)
+		(start 130.775 122.25)
+		(end 126 117.475)
+		(width 0.2)
+		(layer "B.Cu")
+		(net "T3")
+	)
+	(segment
+		(start 126 102.8375)
 		(end 120.0805 96.918)
-		(width 0.2)
-		(layer "B.Cu")
-		(net "T3")
-	)
-	(segment
-		(start 130.775 122.25)
-		(end 128.25 119.725)
 		(width 0.2)
 		(layer "B.Cu")
@@
 	)
 	(segment
-		(start 142.898346 96.918)
-		(end 153.21 86.606346)
+		(start 136.2455 96.918)
+		(end 137.2635 95.9)
+		(width 0.2)
+		(layer "B.Cu")
+		(net "SCL")
+	)
+	(segment
+		(start 151.475686 87.28)
+		(end 152.536346 87.28)
 		(width 0.2)
 		(layer "B.Cu")
@@
 	)
 	(segment
+		(start 137.2635 95.9)
+		(end 142.855686 95.9)
+		(width 0.2)
+		(layer "B.Cu")
+		(net "SCL")
+	)
+	(segment
 		(start 150.67 84.98)
 		(end 149.52 86.13)
@@
 	)
 	(segment
-		(start 136.2455 96.918)
-		(end 142.898346 96.918)
-		(width 0.2)
-		(layer "B.Cu")
-		(net "SCL")
-	)
-	(segment
 		(start 153.21 85.653654)
 		(end 152.536346 84.98)
@@
 	)
 	(segment
+		(start 142.855686 95.9)
+		(end 151.475686 87.28)
+		(width 0.2)
+		(layer "B.Cu")
+		(net "SCL")
+	)
+	(segment
 		(start 153.21 86.606346)
 		(end 153.21 85.653654)
@@
 	)
 	(segment
+		(start 152.536346 87.28)
+		(end 153.21 86.606346)
+		(width 0.2)
+		(layer "B.Cu")
+		(net "SCL")
+	)
+	(segment
+		(start 137.3675 95.5)
+		(end 142.69 95.5)
+		(width 0.2)
+		(layer "B.Cu")
+		(net "SDA")
+	)
+	(segment
+		(start 142.69 95.5)
+		(end 152.06 86.13)
+		(width 0.2)
+		(layer "B.Cu")
+		(net "SDA")
+	)
+	(segment
 		(start 136.2455 94.378)
-		(end 143.812 94.378)
-		(width 0.2)
-		(layer "B.Cu")
-		(net "SDA")
-	)
-	(segment
-		(start 143.812 94.378)
-		(end 152.06 86.13)
-		(width 0.2)
-		(layer "B.Cu")
+		(end 137.3675 95.5)
+		(width 0.2)
+		(layer "B.Cu")
